File: Platine/Hardware.sch (KiCad schematic (older format))
At the start: 158 parts, among them J1 Barrel_Jack, J2 Screw_Terminal_01x02, J3 USB_B, Q1 BCX19, Q2 BCX19, SW1 SW_Soft_Reset, SW2 SW_Hard_Reset, SW3 SW_Flash, U1 ESP32-WROOM-32D, U2 ZLDO1117_SOT223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

Commit message: Finished PCB Layout V1 Updated Inductor for ripple reduction Rerouted FT232RL traces Added reset logic for ISP programming Added Silkscreen button labels
Parts:
- L1: footprint Custom_Footprints:L_1008_2520Metric_Pad1.43x2.20mm_HandSolder -> Inductor_SMD:L_10.4x10.4_H4.8
Changed lines of the file:
@@
 F 0 "L1" V 14840 9200 50  0000 C CNN
 F 1 "33u" V 14749 9200 50  0000 C CNN
-F 2 "Custom_Footprints:L_1008_2520Metric_Pad1.43x2.20mm_HandSolder" H 14650 9200 50  0001 C CNN
+F 2 "Inductor_SMD:L_10.4x10.4_H4.8" H 14650 9200 50  0001 C CNN
 F 3 "https://cdn-reichelt.de/documents/datenblatt/B400/1008F.pdf" H 14650 9200 50  0001 C CNN
 	1    14650 9200

Commit message: Finished review of Layout Reviewed BOM Added input cutoff form screw terminal when barreljack is used Added branding Added revision Added author Optimised routing Added screw holes for case Updated barreljack footprint
Parts:
- removed J1: Barrel_Jack, Connector_BarrelJack:BarrelJack_Horizontal, symbol Connector:Barrel_Jack
- added J1: Barrel_Jack_Switch, Custom_Footprints:BarrelJack_BKL_072759, symbol Connector:Barrel_Jack_Switch
- added TP1: TestPoint 3V3, TestPoint:TestPoint_Pad_D2.0mm, symbol Connector:TestPoint
- added TP2: TestPoint 5V, TestPoint:TestPoint_Pad_D2.0mm, symbol Connector:TestPoint
- added TP3: TestPoint Vin, TestPoint:TestPoint_Pad_D2.0mm, symbol Connector:TestPoint
- added TP4: TestPoint Vusb, TestPoint:TestPoint_Pad_D2.0mm, symbol Connector:TestPoint
- added TP5: TestPoint Vftio, TestPoint:TestPoint_Pad_D2.0mm, symbol Connector:TestPoint
- D44: value D -> B340A
- R43, R44: value 220 -> 300
Connections:
- wire segments 635 -> 646
Other:
- moved on the sheet: C50, J2
Changed lines of the file:
@@
 F 1 "33u" V 14749 9200 50  0000 C CNN
 F 2 "Inductor_SMD:L_10.4x10.4_H4.8" H 14650 9200 50  0001 C CNN
-F 3 "https://cdn-reichelt.de/documents/datenblatt/B400/1008F.pdf" H 14650 9200 50  0001 C CNN
+F 3 "https://cdn-reichelt.de/documents/datenblatt/B400/PIHV4119.pdf" H 14650 9200 50  0001 C CNN
 	1    14650 9200
 	0    -1   -1   0
@@
 P 12000 9400
 F 0 "D44" V 11954 9479 50  0000 L CNN
-F 1 "D" V 12045 9479 50  0000 L CNN
+F 1 "B340A" V 12045 9479 50  0000 L CNN
 F 2 "Diode_SMD:D_SMA_Handsoldering" H 12000 9400 50  0001 C CNN
 F 3 "~" H 12000 9400 50  0001 C CNN
@@
 L Connector:Screw_Terminal_01x02 J2
 U 1 1 5FD151BB
-P 11450 9100
-F 0 "J2" H 11368 8775 50  0000 C CNN
-F 1 "Screw_Terminal_01x02" H 11368 8866 50  0000 C CNN
-F 2 "TerminalBlock_RND:TerminalBlock_RND_205-00001_1x02_P5.00mm_Horizontal" H 11450 9100 50  0001 C CNN
-F 3 "~" H 11450 9100 50  0001 C CNN
-	1    11450 9100
-	-1   0    0    1
-$EndComp
-$Comp
-L Connector:Barrel_Jack J1
-U 1 1 5FD17A0A
-P 11450 9550
-F 0 "J1" H 11507 9875 50  0000 C CNN
-F 1 "Barrel_Jack" H 11507 9784 50  0000 C CNN
-F 2 "Connector_BarrelJack:BarrelJack_Horizontal" H 11500 9510 50  0001 C CNN
-F 3 "~" H 11500 9510 50  0001 C CNN
-	1    11450 9550
-	1    0    0    -1
-$EndComp
-$Comp
-L power:GND #PWR0238
-U 1 1 5FDC5D15
-P 11750 9650
-F 0 "#PWR0238" H 11750 9400 50  0001 C CNN
-F 1 "GND" H 11755 9477 50  0000 C CNN
-F 2 "" H 11750 9650 50  0001 C CNN
-F 3 "" H 11750 9650 50  0001 C CNN
-	1    11750 9650
-	1    0    0    -1
+P 11200 9050
+F 0 "J2" H 11118 8725 50  0000 C CNN
+F 1 "Screw_Terminal_01x02" H 11118 8816 50  0000 C CNN
+F 2 "TerminalBlock_RND:TerminalBlock_RND_205-00001_1x02_P5.00mm_Horizontal" H 11200 9050 50  0001 C CNN
+F 3 "~" H 11200 9050 50  0001 C CNN
+	1    11200 9050
+	0    -1   -1   0
 $EndComp
 $Comp
 L power:GND #PWR0239
 U 1 1 5FDC6D12
-P 11800 9100
-F 0 "#PWR0239" H 11800 8850 50  0001 C CNN
-F 1 "GND" H 11805 8927 50  0000 C CNN
-F 2 "" H 11800 9100 50  0001 C CNN
-F 3 "" H 11800 9100 50  0001 C CNN
-	1    11800 9100
+P 11650 9250
+F 0 "#PWR0239" H 11650 9000 50  0001 C CNN
+F 1 "GND" H 11655 9077 50  0000 C CNN
+F 2 "" H 11650 9250 50  0001 C CNN
+F 3 "" H 11650 9250 50  0001 C CNN
+	1    11650 9250
 	1    0    0    -1
 $EndComp
@@
 	12000 9250 12000 9200
 Wire Wire Line
-	12000 9200 12000 9000
-Wire Wire Line
-	12000 9000 11650 9000
-Connection ~ 12000 9200
-Wire Wire Line
-	11900 9450 11900 9200
-Wire Wire Line
-	11900 9200 12000 9200
-Wire Wire Line
-	11650 9100 11800 9100
-Wire Wire Line
-	11750 9450 11900 9450
-Wire Wire Line
 	12000 9200 12350 9200
 Connection ~ 12350 9200
@@
 P 15250 8100
 F 0 "R43" H 15320 8146 50  0000 L CNN
-F 1 "220" H 15320 8055 50  0000 L CNN
+F 1 "300" H 15320 8055 50  0000 L CNN
 F 2 "Resistor_SMD:R_0805_2012Metric_Pad1.15x1.40mm_HandSolder" V 15180 8100 50  0001 C CNN
 F 3 "~" H 15250 8100 50  0001 C CNN
@@
 P 15650 8100
 F 0 "R44" H 15720 8146 50  0000 L CNN
-F 1 "220" H 15720 8055 50  0000 L CNN
+F 1 "300" H 15720 8055 50  0000 L CNN
 F 2 "Resistor_SMD:R_0805_2012Metric_Pad1.15x1.40mm_HandSolder" V 15580 8100 50  0001 C CNN
 F 3 "~" H 15650 8100 50  0001 C CNN
@@
 Wire Wire Line
 	15650 8300 15650 8250
-$Comp
-L power:GND #PWR0246
-U 1 1 61165DEC
-P 15450 8400
-F 0 "#PWR0246" H 15450 8150 50  0001 C CNN
-F 1 "GND" H 15455 8227 50  0000 C CNN
-F 2 "" H 15450 8400 50  0001 C CNN
-F 3 "" H 15450 8400 50  0001 C CNN
-	1    15450 8400
-	1    0    0    -1
-$EndComp
-Wire Wire Line
-	15450 8400 15450 8300
 Connection ~ 15450 8300
 Wire Wire Line
@@
 L Device:C C50
 U 1 1 63DC313B
-P 12900 5850
-F 0 "C50" H 13015 5896 50  0000 L CNN
-F 1 "100n" H 13015 5805 50  0000 L CNN
-F 2 "Capacitor_SMD:C_0805_2012Metric_Pad1.15x1.40mm_HandSolder" H 12938 5700 50  0001 C CNN
-F 3 "~" H 12900 5850 50  0001 C CNN
-	1    12900 5850
+P 15400 6150
+F 0 "C50" H 15515 6196 50  0000 L CNN
+F 1 "100n" H 15515 6105 50  0000 L CNN
+F 2 "Capacitor_SMD:C_0805_2012Metric_Pad1.15x1.40mm_HandSolder" H 15438 6000 50  0001 C CNN
+F 3 "~" H 15400 6150 50  0001 C CNN
+	1    15400 6150
 	1    0    0    -1
 $EndComp
@@
 Wire Wire Line
 	12750 8000 12550 8000
-Text GLabel 12800 5650 0    50   Input ~ 0
+Text GLabel 15300 5950 0    50   Input ~ 0
 V_FT_IO
 Wire Wire Line
-	12800 5650 12900 5650
+	15300 5950 15400 5950
 Wire Wire Line
-	12900 5650 12900 5700
+	15400 5950 15400 6000
 $Comp
 L power:GND #PWR0251
 U 1 1 641DD522
-P 12900 6000
-F 0 "#PWR0251" H 12900 5750 50  0001 C CNN
-F 1 "GND" H 12905 5827 50  0000 C CNN
-F 2 "" H 12900 6000 50  0001 C CNN
-F 3 "" H 12900 6000 50  0001 C CNN
-	1    12900 6000
+P 15400 6300
+F 0 "#PWR0251" H 15400 6050 50  0001 C CNN
+F 1 "GND" H 15405 6127 50  0000 C CNN
+F 2 "" H 15400 6300 50  0001 C CNN
+F 3 "" H 15400 6300 50  0001 C CNN
+	1    15400 6300
 	1    0    0    -1
 $EndComp
@@
 Text GLabel 11100 5350 2    50   Input ~ 0
 GPIO_0
+$Comp
+L Connector:Barrel_Jack_Switch J1
+U 1 1 5FD5D9CB
+P 11750 8950
+F 0 "J1" V 11761 9130 50  0000 L CNN
+F 1 "Barrel_Jack_Switch" V 11852 9130 50  0000 L CNN
+F 2 "Custom_Footprints:BarrelJack_BKL_072759" H 11800 8910 50  0001 C CNN
+F 3 "https://cdn-reichelt.de/documents/datenblatt/C160/072759.pdf" H 11800 8910 50  0001 C CNN
+	1    11750 8950
+	0    1    1    0
+$EndComp
+Wire Wire Line
+	11750 9250 11750 9550
+Wire Wire Line
+	11750 9550 11300 9550
+Wire Wire Line
+	11300 9250 11300 9550
+Wire Wire Line
+	11200 9250 11200 9600
+Wire Wire Line
+	11200 9600 11850 9600
+Wire Wire Line
+	11850 9600 11850 9300
+Wire Wire Line
+	11850 9300 11950 9300
+Wire Wire Line
+	11950 9300 11950 9200
+Wire Wire Line
+	11950 9200 12000 9200
+Connection ~ 11850 9300
+Wire Wire Line
+	11850 9300 11850 9250
+Connection ~ 12000 9200
+$Comp
+L Connector:TestPoint TP1
+U 1 1 6055D0D0
+P 10900 10500
+F 0 "TP1" H 10958 10618 50  0000 L CNN
+F 1 "TestPoint 3V3" H 10958 10527 50  0000 L CNN
+F 2 "TestPoint:TestPoint_Pad_D2.0mm" H 11100 10500 50  0001 C CNN
+F 3 "~" H 11100 10500 50  0001 C CNN
+	1    10900 10500
+	1    0    0    -1
+$EndComp
+Wire Wire Line
+	10900 10500 10900 10600
+$Comp
+L Connector:TestPoint TP2
+U 1 1 605C9295
+P 15450 9100
+F 0 "TP2" H 15508 9218 50  0000 L CNN
+F 1 "TestPoint 5V" H 15508 9127 50  0000 L CNN
+F 2 "TestPoint:TestPoint_Pad_D2.0mm" H 15650 9100 50  0001 C CNN
+F 3 "~" H 15650 9100 50  0001 C CNN
+	1    15450 9100
+	1    0    0    -1
+$EndComp
+Wire Wire Line
+	15450 9100 15450 9200
+$Comp
+L Connector:TestPoint TP3
+U 1 1 606335C1
+P 12750 9100
+F 0 "TP3" H 12808 9218 50  0000 L CNN
+F 1 "TestPoint Vin" H 12808 9127 50  0000 L CNN
+F 2 "TestPoint:TestPoint_Pad_D2.0mm" H 12950 9100 50  0001 C CNN
+F 3 "~" H 12950 9100 50  0001 C CNN
+	1    12750 9100
+	1    0    0    -1
+$EndComp
+Wire Wire Line
+	12750 9100 12750 9200
+$Comp
+L Connector:TestPoint TP4
+U 1 1 6069F363
+P 12750 7650
+F 0 "TP4" H 12808 7768 50  0000 L CNN
+F 1 "TestPoint Vusb" H 12808 7677 50  0000 L CNN
+F 2 "TestPoint:TestPoint_Pad_D2.0mm" H 12950 7650 50  0001 C CNN
+F 3 "~" H 12950 7650 50  0001 C CNN
+	1    12750 7650
+	1    0    0    -1
+$EndComp
+Wire Wire Line
+	12750 7650 12750 7750
+Connection ~ 12750 7750
+Text GLabel 15400 8450 0    50   Input ~ 0
+V_FT_IO
+Wire Wire Line
+	15400 8450 15450 8450
+Wire Wire Line
+	15450 8300 15450 8450
+$Comp
+L Connector:TestPoint TP5
+U 1 1 6070A6E0
+P 15800 6050
+F 0 "TP5" V 15754 6238 50  0000 L CNN
+F 1 "TestPoint Vftio" V 15845 6238 50  0000 L CNN
+F 2 "TestPoint:TestPoint_Pad_D2.0mm" H 16000 6050 50  0001 C CNN
+F 3 "~" H 16000 6050 50  0001 C CNN
+	1    15800 6050
+	-1   0    0    1
+$EndComp
+Wire Wire Line
+	15800 6050 15800 5950
+Wire Wire Line
+	15800 5950 15400 5950
+Connection ~ 15400 5950
 $EndSCHEMATC
