File: Platine/Hardware.sch (KiCad schematic (older format))
At the start: 170 parts, among them J1 Barrel_Jack_Switch, J2 Screw_Terminal_01x02, J3 USB_B, Q1 BCX19, Q2 BCX19, Q3 DMP3098L7, SW1 SW_Soft_Reset, SW2 SW_Hard_Reset, SW3 SW_Flash, SW4 SW_DPDT_x2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

Commit message: Added Pullup and conneced floating GND peninsulas Added 10k pullup on Soft Rest button (close #9) Via'd GND peninsulas to GND to prevent oscillation
Parts:
- added R52: 10k, Resistor_SMD:R_0805_2012Metric_Pad1.15x1.40mm_HandSolder, symbol Device:R
Connections:
- net IO_S_RST: now also R52.2
- net VCCQ: now also R52.1
Changed lines of the file:
@@
 IO_S_RST
 Wire Wire Line
-	8400 8400 8600 8400
+	8400 8400 8550 8400
 Wire Notes Line
 	500  1200 500  11200
@@
 $EndComp
 $Comp
-L power:GND #PWR?
+L power:GND #PWR0238
 U 1 1 6007E1F7
 P 13500 5250
-F 0 "#PWR?" H 13500 5000 50  0001 C CNN
+F 0 "#PWR0238" H 13500 5000 50  0001 C CNN
 F 1 "GND" H 13505 5077 50  0000 C CNN
 F 2 "" H 13500 5250 50  0001 C CNN
@@
 	13500 4900 13500 5150
 $Comp
-L power:VCCQ #PWR?
+L power:VCCQ #PWR0246
 U 1 1 606D521E
 P 13800 4850
-F 0 "#PWR?" H 13800 4700 50  0001 C CNN
+F 0 "#PWR0246" H 13800 4700 50  0001 C CNN
 F 1 "VCCQ" H 13818 5023 50  0000 C CNN
 F 2 "" H 13800 4850 50  0001 C CNN
@@
 	13800 4750 13850 4750
 $Comp
-L power:VCC #PWR?
+L power:VCC #PWR0252
 U 1 1 60745DA1
 P 14050 4350
-F 0 "#PWR?" H 14050 4200 50  0001 C CNN
+F 0 "#PWR0252" H 14050 4200 50  0001 C CNN
 F 1 "VCC" H 14067 4523 50  0000 C CNN
 F 2 "" H 14050 4350 50  0001 C CNN
@@
 	15000 4950 14950 4950
 $Comp
-L power:VCC #PWR?
+L power:VCC #PWR0253
 U 1 1 60C2B3F3
 P 14950 4300
-F 0 "#PWR?" H 14950 4150 50  0001 C CNN
+F 0 "#PWR0253" H 14950 4150 50  0001 C CNN
 F 1 "VCC" V 14968 4427 50  0000 L CNN
 F 2 "" H 14950 4300 50  0001 C CNN
@@
 Wire Wire Line
 	15050 9200 15050 9300
+$Comp
+L Device:R R52
+U 1 1 603D5712
+P 8550 8100
+F 0 "R52" H 8620 8146 50  0000 L CNN
+F 1 "10k" H 8620 8055 50  0000 L CNN
+F 2 "Resistor_SMD:R_0805_2012Metric_Pad1.15x1.40mm_HandSolder" V 8480 8100 50  0001 C CNN
+F 3 "~" H 8550 8100 50  0001 C CNN
+	1    8550 8100
+	1    0    0    -1
+$EndComp
+Wire Wire Line
+	8600 7850 8550 7850
+Wire Wire Line
+	8550 7850 8550 7950
+Wire Wire Line
+	8550 8250 8550 8400
+Connection ~ 8550 8400
+Wire Wire Line
+	8550 8400 8600 8400
+$Comp
+L power:VCCQ #PWR0254
+U 1 1 604B65AF
+P 8600 7850
+F 0 "#PWR0254" H 8600 7700 50  0001 C CNN
+F 1 "VCCQ" V 8617 7978 50  0000 L CNN
+F 2 "" H 8600 7850 50  0001 C CNN
+F 3 "" H 8600 7850 50  0001 C CNN
+	1    8600 7850
+	0    1    1    0
+$EndComp
 $EndSCHEMATC

Commit message: Switched input smoothing cap to 35V rated cap Switched C3 to 35V rated electrolytic capacitor (close #1)
Parts:
- C3: footprint Capacitor_SMD:CP_Elec_6.3x7.7 -> Capacitor_SMD:CP_Elec_8x10
Changed lines of the file:
@@
 F 0 "C3" H 12468 9396 50  0000 L CNN
 F 1 "470u" H 12468 9305 50  0000 L CNN
-F 2 "Capacitor_SMD:CP_Elec_6.3x7.7" H 12388 9200 50  0001 C CNN
-F 3 "https://cdn-reichelt.de/documents/datenblatt/B300/ABA0000C34.pdf" H 12350 9350 50  0001 C CNN
+F 2 "Capacitor_SMD:CP_Elec_8x10" H 12388 9200 50  0001 C CNN
+F 3 "https://cdn-reichelt.de/documents/datenblatt/B300/MZS.pdf" H 12350 9350 50  0001 C CNN
 	1    12350 9350
 	1    0    0    -1
